Commit message: moved controller parameters from the .xacro file to an independant .yaml file. also updated the code to check that serial is working before trying to send or receive a msg, this prevents it from crashing during this early testing stage.

File: description/ros2_control/rover.ros2_control.xacro (robot description, xacro)
@@ -6,6 +6,8 @@
         <hardware>
           <plugin>mars_rover/RoverSystemHardware</plugin>
-          <param name="serial_port">/dev/ttyUSB0</param>
-          <param name="baud_rate">115200</param>
+          <xacro:property name="yaml_file" value="$(find mars_rover)/config/rover_controller_config.yaml" />
+          <xacro:property name="rover_dict" value="${xacro.load_yaml(yaml_file)}"/>
+          <param name="serial_port">${rover_dict['serial_port']}</param>
+          <param name="baud_rate">${rover_dict['baud_rate']}</param>
         </hardware>
       </xacro:unless>
